File: STM32_schm.kicad_pcb (KiCad board)
At the start: 2 copper layers, 38 x 33.5 mm, 32 parts, among them J1 USB3_B_Micro, J2 Conn_01x04_Pin, J3 Conn_01x04_Pin, J4 Conn_01x04_Pin, SW1 SW_SPDT, U1 STM32F103C8T6, U2 AMS1117-3.3, Y1 16MHz

Commit message: added gerber files
Routing:
- net +3V3: track 160.5 -> 162.0 mm
- net GND: track 38.1 -> 38.9 mm, vias 33 -> 20
Other:
- board text removed: "ON"
Changed lines of the file:
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@@
 		(zone_defaults)
 		(pcbplotparams
-			(layerselection 0x00000000_00000000_55555555_5755f5ff)
+			(layerselection 0x00000000_00000000_55555555_575555ff)
 			(plot_on_all_layers_selection 0x00000000_00000000_00000000_00000000)
 			(disableapertmacros no)
@@
 			(outputformat 1)
 			(mirror no)
-			(drillshape 1)
+			(drillshape 0)
 			(scaleselection 1)
 			(outputdirectory "")
@@
 		(sheetname "/")
 		(sheetfile "STM32_schm.kicad_sch")
-		(units
-			(unit
-				(name "A")
-				(pins "SH" "8" "5" "1" "2" "3" "4" "6" "7" "9" "10")
-			)
-		)
 		(attr smd)
 		(duplicate_pad_numbers_are_jumpers no)
@@
 		)
 		(fp_line
-			(start -3.85 3.3)
-			(end -3.85 3.75)
-			(stroke
-				(width 0.12)
-				(type solid)
-			)
-			(layer "F.SilkS")
-		)
-		(fp_line
 			(start -4.15 3.3)
 			(end -3.85 3.3)
@@
 		)
 		(fp_line
-			(start 3.85 3.75)
-			(end 3.85 3.3)
-			(stroke
-				(width 0.12)
-				(type solid)
-			)
-			(layer "F.SilkS")
-		)
-		(fp_line
 			(start 4.95 -3.34)
 			(end -4.94 -3.34)
@@
 		(tags "capacitor")
 		(property "Reference" "C6"
-			(at -0.5 -1 180)
+			(at -1 -1.5 180)
 			(layer "F.SilkS")
 			(effects
 				(font
-					(size 0.75 0.75)
+					(size 1 1)
 					(thickness 0.15)
 				)
@@
 		(tags "capacitor")
 		(property "Reference" "C13"
-			(at -2.5 -0.5 180)
+			(at -2.85 -1 180)
 			(layer "F.SilkS")
 			(effects
@@
 	)
 	(gr_text "USB"
-		(at 191 96 0)
-		(layer "F.SilkS")
-		(effects
-			(font
-				(size 1 1)
-				(thickness 0.2)
-				(bold yes)
-			)
-			(justify left bottom)
-		)
-	)
-	(gr_text "ON"
-		(at 192 113 0)
+		(at 190.5 96 0)
 		(layer "F.SilkS")
 		(effects
@@
 	)
 	(segment
+		(start 163.52 110.5)
+		(end 163.52 111.48)
+		(width 0.5)
+		(layer "F.Cu")
+		(net "GND")
+	)
+	(segment
 		(start 165.52 106)
 		(end 165 106.52)
@@
 	)
 	(segment
+		(start 163.52 111.48)
+		(end 163.5 111.5)
+		(width 0.5)
+		(layer "F.Cu")
+		(net "GND")
+	)
+	(segment
 		(start 161.096878 107)
 		(end 161.5 107)
@@
 	)
 	(segment
-		(start 163.52 110.5)
-		(end 163.52 111.48)
-		(width 0.3)
-		(layer "F.Cu")
-		(net "GND")
-	)
-	(segment
 		(start 176.16562 103)
 		(end 176.18562 103.02)
@@
 	)
 	(segment
+		(start 168.75 111.5)
+		(end 169.5 111.5)
+		(width 0.5)
+		(layer "F.Cu")
+		(net "GND")
+	)
+	(segment
 		(start 163.780049 105.52)
 		(end 164.12005 105.179999)
@@
 	)
 	(segment
-		(start 163.52 111.48)
-		(end 163.5 111.5)
-		(width 0.3)
-		(layer "F.Cu")
-		(net "GND")
-	)
-	(segment
 		(start 165.69 91)
 		(end 163 91)
@@
 	)
 	(via
-		(at 162.5 109)
-		(size 0.7)
-		(drill 0.3)
-		(layers "F.Cu" "B.Cu")
-		(net "GND")
-	)
-	(via
-		(at 161.5 97)
-		(size 0.7)
-		(drill 0.3)
-		(layers "F.Cu" "B.Cu")
-		(net "GND")
-	)
-	(via
-		(at 175.5 117.5)
-		(size 0.7)
-		(drill 0.3)
-		(layers "F.Cu" "B.Cu")
-		(net "GND")
-	)
-	(via
-		(at 163.5 111.5)
-		(size 0.7)
-		(drill 0.3)
-		(layers "F.Cu" "B.Cu")
-		(net "GND")
-	)
-	(via
 		(at 178.5 103)
 		(size 0.7)
@@
 	)
 	(via
-		(at 176.5 91)
-		(size 0.7)
-		(drill 0.3)
-		(layers "F.Cu" "B.Cu")
-		(net "GND")
-	)
-	(via
 		(at 165 100.5)
 		(size 0.7)
@@
 	)
 	(via
-		(at 163 91)
-		(size 0.7)
-		(drill 0.3)
-		(layers "F.Cu" "B.Cu")
-		(net "GND")
-	)
-	(via
 		(at 186.5 112.5)
 		(size 0.7)
@@
 	)
 	(via
-		(at 173.5 108)
-		(size 0.7)
-		(drill 0.3)
-		(layers "F.Cu" "B.Cu")
-		(net "GND")
-	)
-	(via
-		(at 164.5 103.5)
+		(at 163.5 111.5)
 		(size 0.7)
 		(drill 0.3)
@@
 	)
 	(via
-		(at 178.5 103)
-		(size 0.7)
-		(drill 0.3)
-		(layers "F.Cu" "B.Cu")
-		(net "GND")
-	)
-	(via
 		(at 188.5 111.5)
 		(size 0.7)
@@
 	)
 	(via
-		(at 186.5 99.5)
-		(size 0.7)
-		(drill 0.3)
-		(layers "F.Cu" "B.Cu")
-		(net "GND")
-	)
-	(via
-		(at 169 96)
+		(at 169.5 111.5)
 		(size 0.7)
 		(drill 0.3)
@@
 	)
 	(via
-		(at 164.12005 105.179999)
-		(size 0.7)
-		(drill 0.3)
-		(layers "F.Cu" "B.Cu")
-		(net "GND")
-	)
-	(via
 		(at 185.5 108)
 		(size 0.7)
@@
 	)
 	(via
-		(at 163.5 111.5)
-		(size 0.7)
-		(drill 0.3)
-		(layers "F.Cu" "B.Cu")
-		(net "GND")
-	)
-	(via
-		(at 189.5 110)
-		(size 0.7)
-		(drill 0.3)
-		(layers "F.Cu" "B.Cu")
-		(net "GND")
-	)
-	(via
 		(at 185.5 107)
 		(size 0.7)
@@
 	)
 	(via
-		(at 168.5 106)
-		(size 0.7)
-		(drill 0.3)
-		(layers "F.Cu" "B.Cu")
-		(net "GND")
-	)
-	(via
 		(at 164.12005 105.179999)
 		(size 0.7)
@@
 	)
 	(segment
+		(start 165.7125 110.5)
+		(end 166 110.7875)
+		(width 0.3)
+		(layer "F.Cu")
+		(net "+3V3")
+	)
+	(segment
 		(start 158.55 103.95)
 		(end 160.13 103.95)
@@
 		(start 164.48 110.5)
 		(end 165.7125 110.5)
-		(width 0.5)
+		(width 0.3)
 		(layer "F.Cu")
 		(net "+3V3")
@@
 	)
 	(segment
+		(start 166 109.2125)
+		(end 166 110.7875)
+		(width 0.5)
+		(layer "F.Cu")
+		(net "+3V3")
+	)
+	(segment
 		(start 172.395025 112.635025)
 		(end 173.26 113.5)
@@
 		(width 0.5)
 		(layer "F.Cu")
-		(net "+3V3")
-	)
-	(segment
-		(start 165.7125 110.5)
-		(end 166 110.7875)
-		(width 0.5)
-		(layer "F.Cu")
