File: STM32_schm.kicad_sch (KiCad schematic)
At the start: 32 parts, among them J1 USB3_B_Micro, J2 Conn_01x04_Pin, J3 Conn_01x04_Pin, J4 Conn_01x04_Pin, SW1 SW_SPDT, U1 STM32F103C8T6, U2 AMS1117-3.3, Y1 16MHz

Commit message: added gerber files
Connections:
- net I2C2_SCL: no longer J4.3 (Pin_3), R5.2, U1.22 (PB11)
- new net I2C2_SDA: J4.3 (Pin_3), R5.2, U1.22 (PB11)
Changed lines of the file:
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@@
 		)
 	)
-	(label "I2C2_SCL"
+	(label "I2C2_SDA"
 		(at 125.73 114.3 0)
 		(effects
@@
 		(in_pos_files yes)
 		(dnp no)
-		(fields_autoplaced yes)
 		(property "Reference" "C4"
 			(at 116.84 44.4499 0)
